File: circuits/00-power-supply/schematic/board.kicad_sch (KiCad schematic)
At the start: 0 parts

Commit message: Populate KiCad schematics with real components and global-label nets
Adds Python generator (circuits/tools/gen_kicad.py) that emits self-contained
KiCad v9 schematics with embedded lib_symbols. Each board now contains:

- 00-power-supply: 17 components (LM2596S buck + protection + LEDs + bus header)
- 01-loop-detector: 57 components (4 channels of 2N7000+R+C+LM339+BSS92,
  2x HCF4051 muxes, input/output headers, backplane bus) — verbatim from PDF
- 02-mcu-dspic-sim900: 28 components (dsPIC30F4011 + SIM900 module +
  MP1584 buck + DS1305 RTC + level shifters + ICSP + bus)
- 03-mcu-dspic-air780-w25q80: 34 components (dsPIC + AIR780E + W25Q80 +
  AMS1117 LDO + MP1584 buck + DS1305 + level shifters)
- 04-mcu-stm32-air780-w25q80: 43 components (STM32F103C8 + AIR780E +
  W25Q80 + microSD + crystals + LEDs + SWD + ADC dividers)

All connections expressed as global_labels (no wires drawn) so files are
compact and KiCad can re-route them automatically. Symbol library is inline
(no external KiCad lib install required to open). Re-run the generator to
regenerate after editing.

https://claude.ai/code/session_01FipHdzNRa5m6yYfcuuTEJE
Parts:
- added C1: 470uF/25V, Capacitor_THT:CP_Radial_D10.0mm_P5.00mm, symbol Device:C_Polarized
- added C2: 100nF, Capacitor_SMD:C_0805_2012Metric, symbol Device:C
- added C3: 220uF/10V, Capacitor_SMD:CP_Elec_8x5.4, symbol Device:C_Polarized
- added C4: 10uF, Capacitor_SMD:C_0805_2012Metric, symbol Device:C
- added D1: SS24, Diode_SMD:D_SMA, symbol Device:D
- added D2: SS34, Diode_SMD:D_SMA, symbol Device:D
- added F1: 1A_Polyfuse, Fuse:Fuse_Bourns_MF-RX_TH, symbol Device:R
- added J1: DC_Jack_12V, Connector_BarrelJack:BarrelJack_Horizontal, symbol IVTMS:Conn_1x02
- added J_BUS: Backplane, Connector_PinHeader_2.54mm:PinHeader_2x08_P2.54mm_Vertical, symbol IVTMS:Conn_2x08
- added L1: FB_600R/2A, Inductor_SMD:L_1210_3225Metric, symbol Device:L
- added L2: 33uH/3A, Inductor_SMD:L_Bourns_SRR1280, symbol Device:L
- added LED1: Green, LED_SMD:LED_0805_2012Metric, symbol Device:LED
- added LED2: Red, LED_SMD:LED_0805_2012Metric, symbol Device:LED
- added R1, R2: 1K, Resistor_SMD:R_0805_2012Metric, symbol Device:R
- added TVS1: SMAJ24CA, Diode_SMD:D_SMA, symbol Device:D
- added U1: LM2596S-5.0, Package_TO_SOT_SMD:TO-263-5_TabPin3, symbol IVTMS:LM2596S-5
Other:
- note added: "Input: 12V via J1; Buck: U1 LM2596S-5.0; Output: 5V to backplane"
- note added: "PSU 12V→5V — IVTMS Power Module"
- title: PSU — IVTMS 12V to 5V -> PSU — IVTMS 12V to 5V/2A
