File: circuits/01-loop-detector/schematic/board.kicad_sch (KiCad schematic)
At the start: 0 parts

Commit message: Populate KiCad schematics with real components and global-label nets
Adds Python generator (circuits/tools/gen_kicad.py) that emits self-contained
KiCad v9 schematics with embedded lib_symbols. Each board now contains:

- 00-power-supply: 17 components (LM2596S buck + protection + LEDs + bus header)
- 01-loop-detector: 57 components (4 channels of 2N7000+R+C+LM339+BSS92,
  2x HCF4051 muxes, input/output headers, backplane bus) — verbatim from PDF
- 02-mcu-dspic-sim900: 28 components (dsPIC30F4011 + SIM900 module +
  MP1584 buck + DS1305 RTC + level shifters + ICSP + bus)
- 03-mcu-dspic-air780-w25q80: 34 components (dsPIC + AIR780E + W25Q80 +
  AMS1117 LDO + MP1584 buck + DS1305 + level shifters)
- 04-mcu-stm32-air780-w25q80: 43 components (STM32F103C8 + AIR780E +
  W25Q80 + microSD + crystals + LEDs + SWD + ADC dividers)

All connections expressed as global_labels (no wires drawn) so files are
compact and KiCad can re-route them automatically. Symbol library is inline
(no external KiCad lib install required to open). Re-run the generator to
regenerate after editing.

https://claude.ai/code/session_01FipHdzNRa5m6yYfcuuTEJE
Parts:
- added C11A, C11B, C12A, C12B, C13A, C13B, C14A, C14B: 47nF, Capacitor_SMD:C_0805_2012Metric, symbol Device:C
- added C_BYP_50, C_BYP_51, C_BYP_52: 100nF, Capacitor_SMD:C_0805_2012Metric, symbol Device:C
- added D11A, D12A, D13A, D14A: 1N5819, Diode_SMD:D_SOD-123, symbol Device:D
- added J_BUS: Backplane, Connector_PinHeader_2.54mm:PinHeader_2x08_P2.54mm_Vertical, symbol IVTMS:Conn_2x08
- added P1: Loop_Input, Connector_PinHeader_2.54mm:PinHeader_1x08_P2.54mm_Vertical, symbol IVTMS:Conn_1x08
- added PL: Loop_Output, Connector_PinHeader_2.54mm:PinHeader_1x08_P2.54mm_Vertical, symbol IVTMS:Conn_1x08
- added Q11A, Q11B, Q11C, Q12A, Q12B, Q12C, Q13A, Q13B, Q13C, Q14A, Q14B, Q14C: 2N7000, Package_TO_SOT_SMD:SOT-23, symbol Device:Q_NMOS_GSD
- added Q11D, Q12D, Q13D, Q14D: BSS92, Package_TO_SOT_SMD:SOT-23, symbol Device:Q_PMOS_GSD
- added R11A, R12A, R13A, R14A: 0R, Resistor_SMD:R_0805_2012Metric, symbol Device:R
- added R11B, R12B, R13B, R14B: 10K, Resistor_SMD:R_0805_2012Metric, symbol Device:R
- added R11C, R12C, R13C, R14C: 330K, Resistor_SMD:R_0805_2012Metric, symbol Device:R
- added R11D, R12D, R13D, R14D: 3.3K, Resistor_SMD:R_0805_2012Metric, symbol Device:R
- added R11E, R12E, R13E, R14E: 1K, Resistor_SMD:R_0805_2012Metric, symbol Device:R
- added U50: LM339, Package_SO:SOIC-14_3.9x8.7mm_P1.27mm, symbol IVTMS:LM339
- added U51, U52: HCF4051BEY, Package_SO:SOIC-16_3.9x9.9mm_P1.27mm, symbol IVTMS:HCF4051BEY
Other:
- note added: "Channel 11"
- note added: "Channel 12"
- note added: "Channel 13"
- note added: "Channel 14"
- note added: "LOOP Detector — 4 channels reverse-engineered from main loop pcb3.SchDoc"
- note added: "Note: P1 even pins (loop returns) tie to GND on this board."
- note added: "Per-ch: 2N7000 protect / LM339 quarter / 2SJ196(BSS92) load switch"
- note added: "VTHR = mid-rail reference (from external divider, e.g. 2x10K to VCC/GND)"
- title: LOOP Detector — IVTMS (4-channel) -> LOOP Detector — IVTMS 4-channel
