File: circuits/03-mcu-dspic-air780-w25q80/schematic/board.kicad_sch (KiCad schematic)
At the start: 0 parts

Commit message: Populate KiCad schematics with real components and global-label nets
Adds Python generator (circuits/tools/gen_kicad.py) that emits self-contained
KiCad v9 schematics with embedded lib_symbols. Each board now contains:

- 00-power-supply: 17 components (LM2596S buck + protection + LEDs + bus header)
- 01-loop-detector: 57 components (4 channels of 2N7000+R+C+LM339+BSS92,
  2x HCF4051 muxes, input/output headers, backplane bus) — verbatim from PDF
- 02-mcu-dspic-sim900: 28 components (dsPIC30F4011 + SIM900 module +
  MP1584 buck + DS1305 RTC + level shifters + ICSP + bus)
- 03-mcu-dspic-air780-w25q80: 34 components (dsPIC + AIR780E + W25Q80 +
  AMS1117 LDO + MP1584 buck + DS1305 + level shifters)
- 04-mcu-stm32-air780-w25q80: 43 components (STM32F103C8 + AIR780E +
  W25Q80 + microSD + crystals + LEDs + SWD + ADC dividers)

All connections expressed as global_labels (no wires drawn) so files are
compact and KiCad can re-route them automatically. Symbol library is inline
(no external KiCad lib install required to open). Re-run the generator to
regenerate after editing.

https://claude.ai/code/session_01FipHdzNRa5m6yYfcuuTEJE
Parts:
- added C_BYP_1, C_BYP_2, C_BYP_3, C_BYP_4, C_FLASH_BYP: 100nF, Capacitor_SMD:C_0805_2012Metric, symbol Device:C
- added C_LDO_IN, C_LDO_OUT: 10uF, Capacitor_SMD:C_0805_2012Metric, symbol Device:C
- added C_OSC1, C_OSC2: 22pF, Capacitor_SMD:C_0805_2012Metric, symbol Device:C
- added C_RF_BULK: 470uF/16V, Capacitor_SMD:CP_Elec_8x10.5, symbol Device:C_Polarized
- added D_BUCK: SS34, Diode_SMD:D_SMA, symbol Device:D
- added J_BUS: Backplane, Connector_PinHeader_2.54mm:PinHeader_2x08_P2.54mm_Vertical, symbol IVTMS:Conn_2x08
- added J_ICSP: ICSP, Connector_PinHeader_2.54mm:PinHeader_1x05_P2.54mm_Vertical, symbol IVTMS:Conn_1x05
- added L_BUCK: 10uH, Inductor_SMD:L_Bourns_SRR1280, symbol Device:L
- added R_LVL_MISO, R_LVL_RX: 1K, Resistor_SMD:R_0805_2012Metric, symbol Device:R
- added R_LVL_S0A, R_LVL_S1A, R_LVL_S2A, R_LVL_TX1, R_MCLR, R_PU_PK: 10K, Resistor_SMD:R_0805_2012Metric, symbol Device:R
- added R_LVL_S0B, R_LVL_S1B, R_LVL_S2B: 18K, Resistor_SMD:R_0805_2012Metric, symbol Device:R
- added R_LVL_TX2: 20K, Resistor_SMD:R_0805_2012Metric, symbol Device:R
- added U1: dsPIC30F4011-30I/PT, Package_QFP:TQFP-44_10x10mm_P0.8mm, symbol IVTMS:dsPIC30F4011
- added U2: MP1584EN, Package_SO:SOIC-8_3.9x4.9mm_P1.27mm, symbol IVTMS:MP1584_Buck
- added U3: DS1305, Package_SO:SOIC-16_3.9x9.9mm_P1.27mm, symbol IVTMS:DS1305
- added U4: W25Q80DV, Package_SO:SOIC-8_3.9x4.9mm_P1.27mm, symbol IVTMS:W25Q80
- added U7: AMS1117-3.3, Package_TO_SOT_SMD:SOT-223-3_TabPin2, symbol IVTMS:AMS1117-3.3
- added U8: AIR780E, Module:AIR780E_LCC, symbol IVTMS:AIR780E_Module
- added Y1: 16MHz, Crystal:Crystal_SMD_HC49-SD, symbol Device:Crystal
- added Y2: 32.768kHz, Crystal:Crystal_SMD_3215-2Pin_3.2x1.5mm, symbol Device:Crystal
Other:
- note added: "Buck 12V→3.8V for AIR780, LDO 5V→3.3V for W25Q80 + level shifters"
- note added: "MCU-B: dsPIC30F4011 + AIR780E (4G) + W25Q80 (1MB SPI flash)"
